Commit message: LiDAR 센서와 SLAM을 활용한 MAP 구현

File: src/robot_description/resource/robot.urdf (robot description, URDF)
Before this commit: robot simple_robot, 4 links, 3 joints
Links:
- added link lidar_link, mass 0.3; collision cylinder length=0.07 radius=0.05; visual cylinder length=0.07 radius=0.05
Joints:
- added joint lidar_joint: type fixed, parent base_link, child lidar_link, origin xyz=0.2 0 0.2 rpy=0 0 0
- joint left_wheel_joint: axis 0 0 1 -> 0 0 -1; origin xyz=-0.15 0.24 0 rpy=1.5708 0 0 -> xyz=0.15 0.24 0 rpy=1.5708 0 0
- joint rear_caster_joint: origin xyz=0.2 0 -0.05 rpy=0 0 0 -> xyz=-0.2 0 -0.05 rpy=0 0 0
- joint right_wheel_joint: axis 0 0 1 -> 0 0 -1; origin xyz=-0.15 -0.24 0 rpy=1.5708 0 0 -> xyz=0.15 -0.24 0 rpy=1.5708 0 0
